Commit message: Rebase from 'rpm/jazzy/ur_robot_driver'

File: urdf/ur.ros2_control.xacro (robot description, xacro)
@@ -11,4 +11,5 @@
     input_recipe_filename
     output_recipe_filename
+    ur_type
     transmission_hw_interface:=hardware_interface/PositionJointInterface
     use_mock_hardware:=false mock_sensor_commands:=false
@@ -26,4 +27,5 @@
     robot_receive_timeout:=0.04
     rw_rate:=0
+    verify_robot_model:=false
     ">
     <!-- rw_rate of 0 uses the rate of the controller_manager -->
@@ -48,4 +50,5 @@
           <param name="output_recipe_filename">${output_recipe_filename}</param>
           <param name="input_recipe_filename">${input_recipe_filename}</param>
+          <param name="ur_type">${ur_type}</param>
           <param name="headless_mode">${headless_mode}</param>
           <param name="reverse_port">${reverse_port}</param>
@@ -69,4 +72,5 @@
           <param name="tool_tcp_port">${tool_tcp_port}</param>
           <param name="robot_receive_timeout">${robot_receive_timeout}</param>
+          <param name="verify_robot_model">${verify_robot_model}</param>
         </xacro:unless>
       </hardware>
@@ -162,10 +166,18 @@
         <state_interface name="tool_analog_input_type_0"/>
         <state_interface name="tool_analog_input_type_1"/>
-        <state_interface name="robot_mode"/>
+        <state_interface name="robot_mode">
+          <xacro:if value="${use_mock_hardware}">
+            <param name="initial_value">7</param>
+          </xacro:if>
+        </state_interface>
         <state_interface name="robot_status_bit_0"/>
         <state_interface name="robot_status_bit_1"/>
         <state_interface name="robot_status_bit_2"/>
         <state_interface name="robot_status_bit_3"/>
-        <state_interface name="safety_mode"/>
+        <state_interface name="safety_mode">
+          <xacro:if value="${use_mock_hardware}">
+            <param name="initial_value">1</param>
+          </xacro:if>
+        </state_interface>
         <state_interface name="safety_status_bit_0"/>
         <state_interface name="safety_status_bit_1"/>
@@ -179,5 +191,9 @@
         <state_interface name="safety_status_bit_9"/>
         <state_interface name="safety_status_bit_10"/>
-        <state_interface name="program_running"/>
+        <state_interface name="program_running">
+          <xacro:if value="${use_mock_hardware}">
+            <param name="initial_value">1</param>
+          </xacro:if>
+        </state_interface>
       </gpio>
       <gpio name="${tf_prefix}payload">
@@ -186,5 +202,28 @@
         <command_interface name="cog.y"/>
         <command_interface name="cog.z"/>
+        <command_interface name="inertia.ixx"/>
+        <command_interface name="inertia.iyy"/>
+        <command_interface name="inertia.izz"/>
+        <command_interface name="inertia.ixy"/>
+        <command_interface name="inertia.ixz"/>
+        <command_interface name="inertia.iyz"/>
+        <command_interface name="transition_time"/>
         <command_interface name="payload_async_success"/>
+        <state_interface name="mass"/>
+        <state_interface name="cog.x"/>
+        <state_interface name="cog.y"/>
+        <state_interface name="cog.z"/>
+        <state_interface name="inertia.ixx"/>
+        <state_interface name="inertia.iyy"/>
+        <state_interface name="inertia.izz"/>
+        <state_interface name="inertia.ixy"/>
+        <state_interface name="inertia.ixz"/>
+        <state_interface name="inertia.iyz"/>
+      </gpio>
+      <gpio name="${tf_prefix}gravity">
+        <command_interface name="x"/>
+        <command_interface name="y"/>
+        <command_interface name="z"/>
+        <command_interface name="gravity_async_success"/>
       </gpio>
       <gpio name="${tf_prefix}friction_model">
@@ -283,4 +322,12 @@
         <command_interface name="trajectory_size"/>
       </gpio>
+      <gpio name="${tf_prefix}twist">
+        <command_interface name="linear_velocity_x"/>
+        <command_interface name="linear_velocity_y"/>
+        <command_interface name="linear_velocity_z"/>
+        <command_interface name="angular_velocity_x"/>
+        <command_interface name="angular_velocity_y"/>
+        <command_interface name="angular_velocity_z"/>
+      </gpio>
       <gpio name="${tf_prefix}get_robot_software_version">
         <state_interface name="get_version_major">

File: urdf/ur.urdf.xacro (robot description, xacro)
@@ -31,4 +31,6 @@
   <xacro:arg name="script_sender_port" default="50002"/>
   <xacro:arg name="trajectory_port" default="50003"/>
+  <xacro:arg name="verify_robot_model" default="false" />
+  <xacro:arg name="blocking_read" default="false" />
   <!--   tool communication related parameters-->
   <xacro:arg name="use_tool_communication" default="false" />
@@ -49,4 +51,5 @@
   <!-- convert to property to use substitution in function -->
   <xacro:property name="initial_positions_file" default="$(arg initial_positions_file)"/>
+  <xacro:property name="blocking_read" default="$(arg blocking_read)"/>
   <!-- create link fixed to the "world" -->
   <link name="world" />
@@ -93,4 +96,7 @@
     script_sender_port="$(arg script_sender_port)"
     trajectory_port="$(arg trajectory_port)"
+    ur_type="$(arg ur_type)"
+    verify_robot_model="$(arg verify_robot_model)"
+    non_blocking_read="${not blocking_read}"
   />
 </robot>
