Commit message: Rebase from 'upstream'

File: ur_robot_driver/urdf/ur.ros2_control.xacro (robot description, xacro)
@@ -166,10 +166,18 @@
         <state_interface name="tool_analog_input_type_0"/>
         <state_interface name="tool_analog_input_type_1"/>
-        <state_interface name="robot_mode"/>
+        <state_interface name="robot_mode">
+          <xacro:if value="${use_mock_hardware}">
+            <param name="initial_value">7</param>
+          </xacro:if>
+        </state_interface>
         <state_interface name="robot_status_bit_0"/>
         <state_interface name="robot_status_bit_1"/>
         <state_interface name="robot_status_bit_2"/>
         <state_interface name="robot_status_bit_3"/>
-        <state_interface name="safety_mode"/>
+        <state_interface name="safety_mode">
+          <xacro:if value="${use_mock_hardware}">
+            <param name="initial_value">1</param>
+          </xacro:if>
+        </state_interface>
         <state_interface name="safety_status_bit_0"/>
         <state_interface name="safety_status_bit_1"/>
@@ -183,5 +191,9 @@
         <state_interface name="safety_status_bit_9"/>
         <state_interface name="safety_status_bit_10"/>
-        <state_interface name="program_running"/>
+        <state_interface name="program_running">
+          <xacro:if value="${use_mock_hardware}">
+            <param name="initial_value">1</param>
+          </xacro:if>
+        </state_interface>
       </gpio>
       <gpio name="${tf_prefix}payload">
@@ -190,4 +202,11 @@
         <command_interface name="cog.y"/>
         <command_interface name="cog.z"/>
+        <command_interface name="inertia.ixx"/>
+        <command_interface name="inertia.iyy"/>
+        <command_interface name="inertia.izz"/>
+        <command_interface name="inertia.ixy"/>
+        <command_interface name="inertia.ixz"/>
+        <command_interface name="inertia.iyz"/>
+        <command_interface name="transition_time"/>
         <command_interface name="payload_async_success"/>
         <state_interface name="mass"/>
@@ -195,4 +214,10 @@
         <state_interface name="cog.y"/>
         <state_interface name="cog.z"/>
+        <state_interface name="inertia.ixx"/>
+        <state_interface name="inertia.iyy"/>
+        <state_interface name="inertia.izz"/>
+        <state_interface name="inertia.ixy"/>
+        <state_interface name="inertia.ixz"/>
+        <state_interface name="inertia.iyz"/>
       </gpio>
       <gpio name="${tf_prefix}gravity">
@@ -297,4 +322,12 @@
         <command_interface name="trajectory_size"/>
       </gpio>
+      <gpio name="${tf_prefix}twist">
+        <command_interface name="linear_velocity_x"/>
+        <command_interface name="linear_velocity_y"/>
+        <command_interface name="linear_velocity_z"/>
+        <command_interface name="angular_velocity_x"/>
+        <command_interface name="angular_velocity_y"/>
+        <command_interface name="angular_velocity_z"/>
+      </gpio>
       <gpio name="${tf_prefix}get_robot_software_version">
         <state_interface name="get_version_major">

File: ur_robot_driver/urdf/ur.urdf.xacro (robot description, xacro)
@@ -32,4 +32,5 @@
   <xacro:arg name="trajectory_port" default="50003"/>
   <xacro:arg name="verify_robot_model" default="false" />
+  <xacro:arg name="blocking_read" default="false" />
   <!--   tool communication related parameters-->
   <xacro:arg name="use_tool_communication" default="false" />
@@ -50,4 +51,5 @@
   <!-- convert to property to use substitution in function -->
   <xacro:property name="initial_positions_file" default="$(arg initial_positions_file)"/>
+  <xacro:property name="blocking_read" default="$(arg blocking_read)"/>
   <!-- create link fixed to the "world" -->
   <link name="world" />
@@ -96,4 +98,5 @@
     ur_type="$(arg ur_type)"
     verify_robot_model="$(arg verify_robot_model)"
+    non_blocking_read="${not blocking_read}"
   />
 </robot>

Commit message: Rebase from 'upstream'

File: ur_robot_driver/urdf/ur.ros2_control.xacro (robot description, xacro)
@@ -166,10 +166,18 @@
         <state_interface name="tool_analog_input_type_0"/>
         <state_interface name="tool_analog_input_type_1"/>
-        <state_interface name="robot_mode"/>
+        <state_interface name="robot_mode">
+          <xacro:if value="${use_mock_hardware}">
+            <param name="initial_value">7</param>
+          </xacro:if>
+        </state_interface>
         <state_interface name="robot_status_bit_0"/>
         <state_interface name="robot_status_bit_1"/>
         <state_interface name="robot_status_bit_2"/>
         <state_interface name="robot_status_bit_3"/>
-        <state_interface name="safety_mode"/>
+        <state_interface name="safety_mode">
+          <xacro:if value="${use_mock_hardware}">
+            <param name="initial_value">1</param>
+          </xacro:if>
+        </state_interface>
         <state_interface name="safety_status_bit_0"/>
         <state_interface name="safety_status_bit_1"/>
@@ -183,5 +191,9 @@
         <state_interface name="safety_status_bit_9"/>
         <state_interface name="safety_status_bit_10"/>
-        <state_interface name="program_running"/>
+        <state_interface name="program_running">
+          <xacro:if value="${use_mock_hardware}">
+            <param name="initial_value">1</param>
+          </xacro:if>
+        </state_interface>
       </gpio>
       <gpio name="${tf_prefix}payload">
@@ -310,4 +322,12 @@
         <command_interface name="trajectory_size"/>
       </gpio>
+      <gpio name="${tf_prefix}twist">
+        <command_interface name="linear_velocity_x"/>
+        <command_interface name="linear_velocity_y"/>
+        <command_interface name="linear_velocity_z"/>
+        <command_interface name="angular_velocity_x"/>
+        <command_interface name="angular_velocity_y"/>
+        <command_interface name="angular_velocity_z"/>
+      </gpio>
       <gpio name="${tf_prefix}get_robot_software_version">
         <state_interface name="get_version_major">

File: ur_robot_driver/urdf/ur.urdf.xacro (robot description, xacro)
@@ -32,4 +32,5 @@
   <xacro:arg name="trajectory_port" default="50003"/>
   <xacro:arg name="verify_robot_model" default="true" />
+  <xacro:arg name="blocking_read" default="false" />
   <!--   tool communication related parameters-->
   <xacro:arg name="use_tool_communication" default="false" />
@@ -50,4 +51,5 @@
   <!-- convert to property to use substitution in function -->
   <xacro:property name="initial_positions_file" default="$(arg initial_positions_file)"/>
+  <xacro:property name="blocking_read" default="$(arg blocking_read)"/>
   <!-- create link fixed to the "world" -->
   <link name="world" />
@@ -96,4 +98,5 @@
     ur_type="$(arg ur_type)"
     verify_robot_model="$(arg verify_robot_model)"
+    non_blocking_read="${not blocking_read}"
   />
 </robot>
